File: rocket2-load-cell.kicad_sch (KiCad schematic)
At the start: 45 parts, among them J1 SWD, J3 PJ-002A, J4 Conn_01x02, J5 USB_C_Receptacle_USB2.0_14P, U1 STM32F103C8Tx, U3 LD1117V33, Y1 16MHz

Commit message: Revisions from review. DO NOT USE. please use this as reference since the traces aren't ideal. There are 2 violations (silkscreen clipping) which can easily be fixed and no errors. if you have any more, something is wrong.
Connections:
- net USB_D+: now also J5.A6 (D+)
- net USB_D-: now also J5.A7 (D-)
- no-connect marks 35 -> 33
Changed lines of the file:
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@@
+	)
+	(junction
+		(at 43.18 173.99)
+		(diameter 0)
+		(color 0 0 0 0)
 	)
 	(junction
@@
 	)
 	(no_connect
-		(at 43.18 166.37)
-	)
-	(no_connect
 		(at 124.46 147.32)
 	)
@@
 	(no_connect
 		(at 33.02 119.38)
-	)
-	(no_connect
-		(at 43.18 171.45)
 	)
 	(no_connect
@@
 	(wire
 		(pts
+			(xy 43.18 171.45) (xy 43.18 173.99)
+		)
+		(stroke
+			(width 0)
+			(type default)
+		)
+	)
+	(wire
+		(pts
 			(xy 48.26 173.99) (xy 48.26 181.61)
 		)
@@
 		)
 		(stroke
+			(width 0)
+			(type default)
+		)
+	)
+	(wire
+		(pts
+			(xy 43.18 166.37) (xy 43.18 168.91)
+		)
+		(stroke
