File: rocket2-load-cell.kicad_pcb (KiCad board)
At the start: 2 copper layers, 45 x 90 mm, 47 parts, among them J1 SWD, J3 PJ-002A, J4 Conn_01x02, J5 USB_C_Receptacle_USB2.0_14P, U1 STM32F103C8Tx, U3 LD1117V33, Y1 16MHz

Commit message: LC v1.5 Final Fix
Last Routing Patch for Whole Board
Routing:
- net +3.3V: track 220.9 -> 212.0 mm, vias 4 -> 2
- net USB_VBUS: track 10.5 -> 11.5 mm
- net NRST: track 23.9 -> 23.2 mm
Changed lines of the file:
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@@
-	)
-	(segment
-		(start 132.0375 99.42379)
-		(end 137.27379 99.42379)
-		(width 0.3)
-		(layer "F.Cu")
-		(net 1)
-	)
-	(segment
-		(start 138.951 101.101)
-		(end 138.951 102.33629)
-		(width 0.3)
-		(layer "F.Cu")
-		(net 1)
 	)
 	(segment
@@
 	)
 	(segment
-		(start 137.27379 99.42379)
-		(end 138.951 101.101)
-		(width 0.3)
-		(layer "F.Cu")
-		(net 1)
-	)
-	(segment
 		(start 122 103.7)
 		(end 122 99.48)
@@
 	)
 	(segment
+		(start 143.44879 93.99879)
+		(end 142.37 93.99879)
+		(width 0.2)
+		(layer "F.Cu")
+		(net 1)
+	)
+	(segment
 		(start 133.225 85.475)
 		(end 138.03 85.475)
@@
 	)
 	(segment
+		(start 146.95 97.5)
+		(end 143.44879 93.99879)
+		(width 0.2)
+		(layer "F.Cu")
+		(net 1)
+	)
+	(segment
 		(start 121.51 93.9)
 		(end 121.51121 93.89879)
@@
 	)
 	(segment
-		(start 145.4 95.95)
-		(end 143.44879 93.99879)
-		(width 0.2)
-		(layer "F.Cu")
-		(net 1)
-	)
-	(segment
 		(start 131.14316 99.42379)
 		(end 130.04 100.52695)
@@
 	)
 	(segment
-		(start 143.44879 93.99879)
-		(end 142.37 93.99879)
-		(width 0.2)
-		(layer "F.Cu")
-		(net 1)
-	)
-	(segment
 		(start 131.519999 83.77)
 		(end 129.905 83.77)
 		(width 0.3)
 		(layer "F.Cu")
-		(net 1)
-	)
-	(via
-		(at 145.4 95.95)
-		(size 0.5)
-		(drill 0.2)
-		(layers "F.Cu" "B.Cu")
 		(net 1)
 	)
@@
 		(net 1)
 	)
-	(via
-		(at 146.95 97.5)
-		(size 0.5)
-		(drill 0.2)
-		(layers "F.Cu" "B.Cu")
-		(net 1)
-	)
-	(segment
-		(start 145.4 95.95)
-		(end 146.95 97.5)
-		(width 0.2)
-		(layer "B.Cu")
-		(net 1)
-	)
 	(segment
 		(start 141.2 93.99879)
@@
 	)
 	(segment
+		(start 147.3 92.85)
+		(end 147.44 92.85)
+		(width 0.2)
+		(layer "F.Cu")
+		(net 3)
+	)
+	(segment
+		(start 146.775 93.375)
+		(end 147.3 92.85)
+		(width 0.2)
+		(layer "F.Cu")
+		(net 3)
+	)
+	(segment
 		(start 128.21 98.22379)
 		(end 130.87 98.22379)
@@
 		(start 132.0375 98.42379)
 		(end 136.02379 98.42379)
-		(width 0.2)
-		(layer "F.Cu")
-		(net 3)
-	)
-	(segment
-		(start 146.05 92.85)
-		(end 147.44 92.85)
 		(width 0.2)
 		(layer "F.Cu")
@@
 	)
 	(via
-		(at 146.05 92.85)
+		(at 146.775 93.375)
 		(size 0.5)
 		(drill 0.2)
@@
 	)
 	(segment
-		(start 136.05 98.45)
+		(start 146.775 93.375)
 		(end 141.7 98.45)
 		(width 0.2)
@@
 	)
 	(segment
-		(start 146.05 94.1)
-		(end 146.05 92.85)
-		(width 0.2)
-		(layer "B.Cu")
-		(net 3)
-	)
-	(segment
-		(start 141.775 98.375)
-		(end 146.05 94.1)
-		(width 0.2)
-		(layer "B.Cu")
-		(net 3)
-	)
-	(segment
 		(start 141.7 98.45)
-		(end 141.775 98.375)
+		(end 136.05 98.45)
 		(width 0.2)
 		(layer "B.Cu")
@@
 	)
 	(segment
-		(start 148.549135 106.150865)
-		(end 148.549135 106.135034)
+		(start 145.2 109.5)
+		(end 145.2 107.7)
 		(width 0.2)
 		(layer "B.Cu")
@@
 	)
 	(segment
-		(start 145.2 109.5)
-		(end 148.549135 106.150865)
+		(start 145.2 107.7)
+		(end 146.764966 106.135034)
 		(width 0.2)
 		(layer "B.Cu")
+		(net 6)
+	)
+	(segment
+		(start 146.764966 106.135034)
+		(end 148.549135 106.135034)
+		(width 0.2)
+		(layer "B.Cu")
